File: kicad/egdab.sch (KiCad schematic (older format))
At the start: 10 parts

Commit message: Schematic WIP
Parts:
- removed SW?: SW_Push, symbol Switch:SW_Push
- removed U?: MAN71A, Display_7Segment:MAN71A, symbol Display_Character:MAN71A
- added BT?: Battery_Cell, symbol Device:Battery_Cell
- added J?: Conn_02x10_Counter_Clockwise, symbol Connector_Generic:Conn_02x10_Counter_Clockwise
- added R? (x17): R, symbol Device:R
- added RV? (x4): R_POT, symbol Device:R_POT
- added SW? (x2): SW_Push, symbol Switch:SW_Push
- added SW?: SW_DIP_x12, symbol Switch:SW_DIP_x12
- added U?: BU2506FV, MODULE, symbol BU2506FV:BU2506FV
- added U?: LM35-D, Package_SO:SOIC-8_3.9x4.9mm_P1.27mm, symbol Sensor_Temperature:LM35-D
- added U?: MAX7221, symbol smisoto-w_logic:MAX7221
- added U?: 74165, symbol 74xx_IEEE:74165
- added U? (x3): HDSP-A151, Display_7Segment:HDSP-A151, symbol Display_Character:HDSP-A151
- added U?: 74HC4316, MODULE, symbol 74HC4316:74HC4316
Connections:
- net labels added: +5V, GND, INPUT_SR, INPUT_SR_CLK, INPUT_SR_SH
- wire segments 0 -> 317
Other:
- note added: "TODO\n\n- power conditioning capacitors\n- touch capacitance capacitors (?)\n- MAX7221 data connection\n- DAC data connection\n- header: spi, programmer, i2c?, dac, sensor"
- moved on the sheet: MK?, SW?

Commit message: Global labels
Parts:
- added U?: AS1115-BSST, Package_SO:QSOP-24_3.9x8.7mm_P0.635mm, symbol Interface_Expansion:AS1115-BSST
Connections:
- net labels added: DAC_CLK, DAC_DI, DAC_LD, MULT_1, MULT_2, MULT_3, MULT_4, MULT_E
- wire segments 317 -> 324
Other:
- note added: "TODO\n\n- power conditioning capacitors\n- MAX7221 data connection\n- DAC data connection\n- header: spi, programmer, i2c?, dac, sensor"
- note added: "TODO\n\nReplace MAX7221 and 2x shift registers with AS1115"
- note removed: "TODO\n\n- power conditioning capacitors\n- touch capacitance capacitors (?)\n- MAX7221 data connection\n- DAC data connection\n- header: spi, programmer, i2c?, dac, sensor"
Changed lines of the file:
@@
 L MCU_Microchip_ATmega:ATmega328P-AU U?
 U 1 1 5D0758F5
-P 2700 3350
-F 0 "U?" H 2700 1761 50  0000 C CNN
-F 1 "ATmega328P-AU" H 2700 1670 50  0000 C CNN
-F 2 "Package_QFP:TQFP-32_7x7mm_P0.8mm" H 2700 3350 50  0001 C CIN
-F 3 "http://ww1.microchip.com/downloads/en/DeviceDoc/ATmega328_P%20AVR%20MCU%20with%20picoPower%20Technology%20Data%20Sheet%2040001984A.pdf" H 2700 3350 50  0001 C CNN
-	1    2700 3350
+P 1600 2400
+F 0 "U?" H 1600 811 50  0000 C CNN
+F 1 "ATmega328P-AU" H 1600 720 50  0000 C CNN
+F 2 "Package_QFP:TQFP-32_7x7mm_P0.8mm" H 1600 2400 50  0001 C CIN
+F 3 "http://ww1.microchip.com/downloads/en/DeviceDoc/ATmega328_P%20AVR%20MCU%20with%20picoPower%20Technology%20Data%20Sheet%2040001984A.pdf" H 1600 2400 50  0001 C CNN
+	1    1600 2400
 	1    0    0    -1
 $EndComp
@@
 	14750 1150 14850 1150
 Text Notes 5750 2400 0    138  ~ 0
-TODO\n\n- power conditioning capacitors\n- touch capacitance capacitors (?)\n- MAX7221 data connection\n- DAC data connection\n- header: spi, programmer, i2c?, dac, sensor
+TODO\n\n- power conditioning capacitors\n- MAX7221 data connection\n- DAC data connection\n- header: spi, programmer, i2c?, dac, sensor
 $Comp
 L Device:R_POT RV?
@@
 	1    0    0    -1
 $EndComp
+Text GLabel 6350 4650 0    50   Input ~ 0
+MULT_E
+Text GLabel 6350 4850 0    50   Input ~ 0
+MULT_1
+Text GLabel 6350 5050 0    50   Input ~ 0
+MULT_2
+Text GLabel 6350 5250 0    50   Input ~ 0
+MULT_3
+Text GLabel 6350 5450 0    50   Input ~ 0
+MULT_4
+Text GLabel 3750 2950 2    50   Input ~ 0
+MULT_E
+Text GLabel 2800 2100 2    50   Input ~ 0
+MULT_1
+Text GLabel 2800 2200 2    50   Input ~ 0
+MULT_2
+Text GLabel 2800 2300 2    50   Input ~ 0
+MULT_3
+Text GLabel 2800 2400 2    50   Input ~ 0
+MULT_4
+Wire Wire Line
+	2800 2100 2200 2100
+Wire Wire Line
+	2200 2200 2800 2200
+Wire Wire Line
+	2800 2300 2200 2300
+Wire Wire Line
+	2200 2400 2800 2400
+Text GLabel 3250 3500 2    50   Input ~ 0
+INPUT_SR_SH
+Text GLabel 3250 3750 2    50   Input ~ 0
+INPUT_SR_CLK
+Text GLabel 3250 4000 2    50   Input ~ 0
+INPUT_SR
+Text GLabel 3850 10600 0    50   Input ~ 0
+DAC_DI
+Text GLabel 3850 10800 0    50   Input ~ 0
+DAC_LD
+Text GLabel 3850 10700 0    50   Input ~ 0
+DAC_CLK
+Wire Wire Line
+	3850 10600 4200 10600
+Wire Wire Line
+	4200 10700 3850 10700
+Wire Wire Line
+	3850 10800 4200 10800
+Text GLabel 3300 4450 2    50   Input ~ 0
+DAC_DI
+Text GLabel 3300 4650 2    50   Input ~ 0
+DAC_LD
+Text GLabel 3300 4550 2    50   Input ~ 0
+DAC_CLK
+$Comp
+L Interface_Expansion:AS1115-BSST U?
+U 1 1 5D451D3E
+P -3500 6150
+F 0 "U?" H -3500 7531 50  0000 C CNN
+F 1 "AS1115-BSST" H -3500 7440 50  0000 C CNN
+F 2 "Package_SO:QSOP-24_3.9x8.7mm_P0.635mm" H -3500 6150 50  0001 C CNN
+F 3 "https://ams.com/documents/20143/36005/AS1115_DS000206_1-00.pdf/3d3e6d35-b184-1329-adf9-2d769eb2404f" H -3500 6150 50  0001 C CNN
+	1    -3500 6150
+	1    0    0    -1
+$EndComp
+Text Notes -4150 4150 0    50   ~ 0
+TODO\n\nReplace MAX7221 and 2x shift registers with AS1115
 $EndSCHEMATC

Commit message: AS1115 takeover, needs diodes for keyscan
Parts:
- removed D? (x3): LED_CRGB, symbol Device:LED_CRGB
- removed R? (x17): R, symbol Device:R
- removed SW? (x4): SW_Push, symbol Switch:SW_Push
- removed SW?: SW_DIP_x12, symbol Switch:SW_DIP_x12
- removed U?: BU2506FV, MODULE, symbol BU2506FV:BU2506FV
- removed U?: MAX7221, symbol smisoto-w_logic:MAX7221
- removed U? (x2): 74165, symbol 74xx_IEEE:74165
- removed U?: HDSP-A151, Display_7Segment:HDSP-A151, symbol Display_Character:HDSP-A151
- added D? (x6): LED_RGB, symbol Device:LED_RGB
- added D? (x16): D, symbol Device:D
- added SW? (x4): SW_Push, symbol Switch:SW_Push
- added SW?: SW_DIP_x12, symbol Switch:SW_DIP_x12
Connections:
- net labels added: AS1115_IRQ, AS1115_ISET, AS1115_SCL, AS1115_SDA
- net labels removed: DAC_CLK, DAC_DI, DAC_LD, INPUT_SR, INPUT_SR_CLK, INPUT_SR_SH
- wire segments 324 -> 229
Other:
- note removed: "TODO\n\nReplace MAX7221 and 2x shift registers with AS1115"
- moved on the sheet: U?

Commit message: ATtiny1606 instead of Atmega328p
Parts:
- removed MK?: Microphone, symbol Device:Microphone
- removed RV? (x4): R_POT, symbol Device:R_POT
- removed U?: LM35-D, Package_SO:SOIC-8_3.9x4.9mm_P1.27mm, symbol Sensor_Temperature:LM35-D
- removed U?: ATmega328P-AU, Package_QFP:TQFP-32_7x7mm_P0.8mm, symbol MCU_Microchip_ATmega:ATmega328P-AU
- removed U?: 74HC4316, MODULE, symbol 74HC4316:74HC4316
- added MK?: Microphone, symbol Device:Microphone
- added R?: R, symbol Device:R
- added RV? (x5): R_POT, symbol Device:R_POT
- added U?: ATtiny1606-S, Package_SO:SOIC-20W_7.5x12.8mm_P1.27mm, symbol MCU_Microchip_ATtiny:ATtiny1606-S
- added U?: LM35-D, Package_SO:SOIC-8_3.9x4.9mm_P1.27mm, symbol Sensor_Temperature:LM35-D
Connections:
- net labels added: PB2, PB3, SPI_MISO, SPI_MOSI, SPI_SCK, SPI_SS
- net labels removed: AS1115_ISET, MULT_1, MULT_2, MULT_3, MULT_4, MULT_E
- wire segments 229 -> 297
Other:
- note added: "TODO to VDD or RSET resistor"
- note added: "TODO\n- power conditioning capacitors\n- header: spi, programmer, i2c?, dac, sensor\n- as1115 brightness\n- microphone circuit"
- note removed: "TODO\n\n- power conditioning capacitors\n- MAX7221 data connection\n- DAC data connection\n- header: spi, programmer, i2c?, dac, sensor"
- moved on the sheet: BT?, D?, J?, SW?, U?

Commit message: First draft of schematic
Parts:
- removed J?: Conn_02x10_Counter_Clockwise, symbol Connector_Generic:Conn_02x10_Counter_Clockwise
- removed MK?: Microphone, symbol Device:Microphone
- added C? (x8): 22uF, symbol Device:C
- added C? (x4): 10uF, symbol Device:C
- added J?: AudioJack2, symbol Connector:AudioJack2
- added J?: Conn_02x03_Counter_Clockwise, symbol Connector_Generic:Conn_02x03_Counter_Clockwise
- added J?: Conn_02x10_Counter_Clockwise, symbol Connector_Generic:Conn_02x10_Counter_Clockwise
- added MK?: Microphone, symbol Device:Microphone
- added R?: 22K, symbol Device:R
- added R? (x8): 10K, symbol Device:R
- added U?: CAP1296, Package_SO:SOIC-14_3.9x8.7mm_P1.27mm, symbol Sensor_Touch:CAP1206-x-SL
- BT?: value Battery_Cell -> CR2450VP
- R?: value R -> 10K
Connections:
- net labels added: +3V0, I2C_SCL, I2C_SDA, RESET, TOUCH1, TOUCH2, TOUCH_GUARD, TOUCH_PROX, UI_INTERRUPT
- net labels removed: +5V, AS1115_IRQ, AS1115_SCL, AS1115_SDA, touch
- wire segments 297 -> 445
Other:
- note removed: "TODO to VDD or RSET resistor"
- moved on the sheet: BT?, D?, R?, RV?, SW?, U?

Commit message: PCB WIP
Parts:
- BT1: renamed from BT?; footprint (none) -> Battery_Holders:Keystone_3008_1x2450-CoinCell
- C1, C10, C11, C12, C2, C3, C4, C5, C6, C7, C8, C9: renamed from C?; footprint (none) -> Capacitors_SMD:C_0603_HandSoldering
- D1, D12, D13, D16, D17, D19, D2, D21, D22, D3, D4, D5, D6, D7, D8, D9: renamed from D?; footprint (none) -> Diodes_SMD:D_SOD-523
- D10, D11, D14, D15, D18, D20: renamed from D?; footprint (none) -> LEDs:LED_RGB_PLCC-6
- J2: renamed from J?; footprint (none) -> Pin_Headers:Pin_Header_Straight_2x03_Pitch2.54mm
- J3: renamed from J?; footprint (none) -> Pin_Headers:Pin_Header_Angled_2x10_Pitch2.54mm
- R1, R10, R2, R3, R4, R5, R6, R7, R8, R9: renamed from R?; footprint (none) -> Resistors_SMD:R_0603_HandSoldering
- RV1, RV2, RV3, RV4, RV5: renamed from RV?; footprint (none) -> Potentiometers:Potentiometer_Trimmer_Suntan_TSR-3386P_Horizontal
- SW1: renamed from SW?; footprint (none) -> Buttons_Switches_SMD:SW_DIP_x12_W8.61mm_Slide_LowProfile
- U1: renamed from U?; footprint Package_SO:SOIC-20W_7.5x12.8mm_P1.27mm -> Housings_SOIC:SOIC-20W_7.5x12.8mm_Pitch1.27mm
- U2: renamed from U?; footprint Package_SO:QSOP-24_3.9x8.7mm_P0.635mm -> Housings_SSOP:SSOP-24_3.9x8.7mm_Pitch0.635mm
- U3: renamed from U?; footprint Package_SO:SOIC-8_3.9x4.9mm_P1.27mm -> Housings_SOIC:SOIC-8_3.9x4.9mm_Pitch1.27mm
- U4: renamed from U?; footprint Package_SO:SOIC-14_3.9x8.7mm_P1.27mm -> Housings_SOIC:SOIC-14_3.9x8.7mm_Pitch1.27mm
- gave numbers to parts that had none: 8
Connections:
- wire segments 445 -> 446
Other:
- note added: "TODO share voltage divider and capacitor between audio sources"

Commit message: Big things
Parts:
- removed C12: 10uF, Capacitors_SMD:C_0603_HandSoldering, symbol Device:C
- removed J3: Conn_02x10_Counter_Clockwise, Pin_Headers:Pin_Header_Angled_2x10_Pitch2.54mm, symbol Connector_Generic:Conn_02x10_Counter_Clockwise
- removed R8, R9: 10K, Resistors_SMD:R_0603_HandSoldering, symbol Device:R
- removed U5, U6: HDSP-A151, Display_7Segment:HDSP-A151, symbol Display_Character:HDSP-A151
- added D23: 7SegmentLED_ACDA02, BBS Components:7SegmentLED_ACDA02, symbol egdab:7SegmentLED_ACDA02
- added D24: LED_RGB, LEDs:LED_RGB_PLCC-6, symbol Device:LED_RGB
- added J3: Conn_02x04_Counter_Clockwise, BBS Components:Header_SMD_vertical_passthrough_02x04, symbol Connector_Generic:Conn_02x04_Counter_Clockwise
- added SW6: SW_SPST, symbol Switch:SW_SPST
- J2: footprint Pin_Headers:Pin_Header_Straight_2x03_Pitch2.54mm -> BBS Components:Header_SMD_vertical_passthrough_02x03
- SW2, SW3, SW4, SW5: footprint (none) -> BBS Components:SW_SPST_SMD_3_6
Connections:
- net labels added: AS1115_ISET, AUDIO, DIG0, DIG1, DIG2, DIG3, DIG4, DIG5, DIG6, DIG7, KEYA, KEYB, MIC, POT1, POT2, POT3, POT4, POT5, SEGA, SEGB, SEGC, SEGD, SEGDP, SEGE, SEGF, SEGG, TEMP
- wire segments 446 -> 489
Other:
- note removed: "TODO\n- power conditioning capacitors\n- header: spi, programmer, i2c?, dac, sensor\n- as1115 brightness\n- microphone circuit"
- moved on the sheet: D10, D11, D14, D15, D18, D20, R1

Commit message: PCB layout progress
Parts:
- SW6: footprint (none) -> Digikey:Switch_Slide_JS202011SCQN
Connections:
- net labels added: BAT+
- wire segments 489 -> 505
