File: kicad/egdab.sch (KiCad schematic (older format))
At the start: 63 parts, among them J1 AudioJack2, J2 Conn_02x03_Counter_Clockwise, J3 Conn_02x04_Counter_Clockwise, SW1 SW_DIP_x12, SW2 SW_Push, SW3 SW_Push, SW4 SW_Push, SW5 SW_Push, SW6 SW_SPST, U1 ATtiny1606-S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

Commit message: Draft 1 may be complete
Parts:
- removed J1: AudioJack2, symbol Connector:AudioJack2
- added J1: Audio-Jack-2_Switch, BBS Components:sj2-35852b-smt, symbol synthrotek2:Audio-Jack-2_Switch
- MK1: footprint (none) -> BBS Components:spv1840l45h-b
Changed lines of the file:
@@
 F 0 "MK1" H 9280 996 50  0000 L CNN
 F 1 "Microphone" H 9280 905 50  0000 L CNN
-F 2 "" V 9150 1050 50  0001 C CNN
+F 2 "BBS Components:spv1840l45h-b" V 9150 1050 50  0001 C CNN
 F 3 "~" V 9150 1050 50  0001 C CNN
 	1    9150 950
@@
 	1    7850 2450
 	1    0    0    -1
-$EndComp
-Wire Wire Line
-	7750 3300 7850 3300
-Wire Wire Line
-	7750 1150 7750 3300
-$Comp
-L Connector:AudioJack2 J1
-U 1 1 5F657110
-P 7850 950
-F 0 "J1" V 7836 1138 50  0000 L CNN
-F 1 "AudioJack2" V 7927 1138 50  0000 L CNN
-F 2 "" H 7850 950 50  0001 C CNN
-F 3 "~" H 7850 950 50  0001 C CNN
-	1    7850 950
-	0    -1   1    0
 $EndComp
 Wire Wire Line
@@
 Text Label 850  10000 0    50   ~ 0
 BAT+
+$Comp
+L synthrotek2:Audio-Jack-2_Switch J1
+U 1 1 5D7366F8
+P 7750 950
+F 0 "J1" V 7682 1138 50  0000 L CNN
+F 1 "Audio-Jack-2_Switch" V 7773 1138 50  0000 L CNN
+F 2 "BBS Components:sj2-35852b-smt" H 8000 1050 50  0001 C CNN
+F 3 "~" H 8000 1050 50  0001 C CNN
+	1    7750 950
+	0    1    1    0
+$EndComp
+Wire Wire Line
+	7650 750  7650 3300
+Wire Wire Line
+	7650 3300 7850 3300
 $EndSCHEMATC

Commit message: Moar
Parts:
- D10, D11, D14, D15, D18, D20, D24: footprint LEDs:LED_RGB_PLCC-6 -> BBS Components:plcc_6_reverse_smd_rgb_led
Changed lines of the file:
@@
 F 0 "D15" V 11196 8970 50  0000 R CNN
 F 1 "LED_RGB" V 11105 8970 50  0000 R CNN
-F 2 "LEDs:LED_RGB_PLCC-6" H 11150 9250 50  0001 C CNN
+F 2 "BBS Components:plcc_6_reverse_smd_rgb_led" H 11150 9250 50  0001 C CNN
 F 3 "~" H 11150 9250 50  0001 C CNN
 	1    11150 9300
@@
 F 0 "D11" V 10146 8970 50  0000 R CNN
 F 1 "LED_RGB" V 10055 8970 50  0000 R CNN
-F 2 "LEDs:LED_RGB_PLCC-6" H 10100 9250 50  0001 C CNN
+F 2 "BBS Components:plcc_6_reverse_smd_rgb_led" H 10100 9250 50  0001 C CNN
 F 3 "~" H 10100 9250 50  0001 C CNN
 	1    10100 9300
@@
 F 0 "D20" V 11196 10070 50  0000 R CNN
 F 1 "LED_RGB" V 11105 10070 50  0000 R CNN
-F 2 "LEDs:LED_RGB_PLCC-6" H 11150 10350 50  0001 C CNN
+F 2 "BBS Components:plcc_6_reverse_smd_rgb_led" H 11150 10350 50  0001 C CNN
 F 3 "~" H 11150 10350 50  0001 C CNN
 	1    11150 10400
@@
 F 0 "D18" V 10146 10070 50  0000 R CNN
 F 1 "LED_RGB" V 10055 10070 50  0000 R CNN
-F 2 "LEDs:LED_RGB_PLCC-6" H 10100 10350 50  0001 C CNN
+F 2 "BBS Components:plcc_6_reverse_smd_rgb_led" H 10100 10350 50  0001 C CNN
 F 3 "~" H 10100 10350 50  0001 C CNN
 	1    10100 10400
@@
 F 0 "D14" V 10846 7870 50  0000 R CNN
 F 1 "LED_RGB" V 10755 7870 50  0000 R CNN
-F 2 "LEDs:LED_RGB_PLCC-6" H 10800 8150 50  0001 C CNN
+F 2 "BBS Components:plcc_6_reverse_smd_rgb_led" H 10800 8150 50  0001 C CNN
 F 3 "~" H 10800 8150 50  0001 C CNN
 	1    10800 8200
@@
 F 0 "D10" V 11546 7870 50  0000 R CNN
 F 1 "LED_RGB" V 11455 7870 50  0000 R CNN
-F 2 "LEDs:LED_RGB_PLCC-6" H 11500 8150 50  0001 C CNN
+F 2 "BBS Components:plcc_6_reverse_smd_rgb_led" H 11500 8150 50  0001 C CNN
 F 3 "~" H 11500 8150 50  0001 C CNN
 	1    11500 8200
@@
 F 0 "D24" V 10146 7870 50  0000 R CNN
 F 1 "LED_RGB" V 10055 7870 50  0000 R CNN
-F 2 "LEDs:LED_RGB_PLCC-6" H 10100 8150 50  0001 C CNN
+F 2 "BBS Components:plcc_6_reverse_smd_rgb_led" H 10100 8150 50  0001 C CNN
 F 3 "~" H 10100 8150 50  0001 C CNN
 	1    10100 8200

Commit message: v2 PCB in progress
- board version added to silk
- use actual reverse mount RGB LEDs
- invert lower petal soldermask
Parts:
- D10, D11, D14, D15, D18, D20, D24: footprint BBS Components:plcc_6_reverse_smd_rgb_led -> BBS Components:LED_RGB_SMD_PLCC4_Reverse_XZMDKCBDDG45S; symbol Device:LED_RGB -> Device:LED_BARG
Connections:
- net labels added: ALL_SEG
- wire segments 505 -> 477
Changed lines of the file:
@@
 Wire Wire Line
 	15600 6700 15600 9450
-$Comp
-L Device:LED_RGB D15
-U 1 1 5E6D21EF
-P 11150 9300
-F 0 "D15" V 11196 8970 50  0000 R CNN
-F 1 "LED_RGB" V 11105 8970 50  0000 R CNN
-F 2 "BBS Components:plcc_6_reverse_smd_rgb_led" H 11150 9250 50  0001 C CNN
-F 3 "~" H 11150 9250 50  0001 C CNN
-	1    11150 9300
-	0    -1   1    0
-$EndComp
-$Comp
-L Device:LED_RGB D11
-U 1 1 5E7108CE
-P 10100 9300
-F 0 "D11" V 10146 8970 50  0000 R CNN
-F 1 "LED_RGB" V 10055 8970 50  0000 R CNN
-F 2 "BBS Components:plcc_6_reverse_smd_rgb_led" H 10100 9250 50  0001 C CNN
-F 3 "~" H 10100 9250 50  0001 C CNN
-	1    10100 9300
-	0    -1   1    0
-$EndComp
-$Comp
-L Device:LED_RGB D20
-U 1 1 5E72EAEB
-P 11150 10400
-F 0 "D20" V 11196 10070 50  0000 R CNN
-F 1 "LED_RGB" V 11105 10070 50  0000 R CNN
-F 2 "BBS Components:plcc_6_reverse_smd_rgb_led" H 11150 10350 50  0001 C CNN
-F 3 "~" H 11150 10350 50  0001 C CNN
-	1    11150 10400
-	0    -1   1    0
-$EndComp
-$Comp
-L Device:LED_RGB D18
-U 1 1 5E789449
-P 10100 10400
-F 0 "D18" V 10146 10070 50  0000 R CNN
-F 1 "LED_RGB" V 10055 10070 50  0000 R CNN
-F 2 "BBS Components:plcc_6_reverse_smd_rgb_led" H 10100 10350 50  0001 C CNN
-F 3 "~" H 10100 10350 50  0001 C CNN
-	1    10100 10400
-	0    -1   1    0
-$EndComp
-$Comp
-L Device:LED_RGB D14
-U 1 1 5E7D3281
-P 10800 8200
-F 0 "D14" V 10846 7870 50  0000 R CNN
-F 1 "LED_RGB" V 10755 7870 50  0000 R CNN
-F 2 "BBS Components:plcc_6_reverse_smd_rgb_led" H 10800 8150 50  0001 C CNN
-F 3 "~" H 10800 8150 50  0001 C CNN
-	1    10800 8200
-	0    -1   1    0
-$EndComp
-$Comp
-L Device:LED_RGB D10
-U 1 1 5E7D3287
-P 11500 8200
-F 0 "D10" V 11546 7870 50  0000 R CNN
-F 1 "LED_RGB" V 11455 7870 50  0000 R CNN
-F 2 "BBS Components:plcc_6_reverse_smd_rgb_led" H 11500 8150 50  0001 C CNN
-F 3 "~" H 11500 8150 50  0001 C CNN
-	1    11500 8200
-	0    -1   1    0
-$EndComp
 Wire Wire Line
 	4250 7200 9600 7200
@@
 Wire Wire Line
 	2600 6600 3050 6600
-$Comp
-L Device:LED_RGB D24
-U 1 1 5DC39FA4
-P 10100 8200
-F 0 "D24" V 10146 7870 50  0000 R CNN
-F 1 "LED_RGB" V 10055 7870 50  0000 R CNN
-F 2 "BBS Components:plcc_6_reverse_smd_rgb_led" H 10100 8150 50  0001 C CNN
-F 3 "~" H 10100 8150 50  0001 C CNN
-	1    10100 8200
-	0    -1   1    0
-$EndComp
 Wire Wire Line
 	11850 7450 11850 8550
@@
 Wire Wire Line
 	9900 7850 10600 7850
-Wire Wire Line
-	11700 8400 11700 8550
-Wire Wire Line
-	11700 8550 11850 8550
 Connection ~ 11850 8550
-Wire Wire Line
-	11700 8550 11500 8550
-Wire Wire Line
-	9900 8550 9900 8400
-Connection ~ 11700 8550
-Wire Wire Line
-	10100 8400 10100 8550
-Connection ~ 10100 8550
-Wire Wire Line
-	10100 8550 9900 8550
-Wire Wire Line
-	10300 8400 10300 8550
-Connection ~ 10300 8550
-Wire Wire Line
-	10300 8550 10100 8550
-Wire Wire Line
-	10600 8400 10600 8550
-Connection ~ 10600 8550
-Wire Wire Line
-	10600 8550 10300 8550
 Wire Wire Line
 	10800 8400 10800 8550
 Connection ~ 10800 8550
 Wire Wire Line
-	10800 8550 10600 8550
-Wire Wire Line
-	11000 8400 11000 8550
-Connection ~ 11000 8550
-Wire Wire Line
-	11000 8550 10800 8550
-Wire Wire Line
-	11300 8400 11300 8550
-Connection ~ 11300 8550
-Wire Wire Line
-	11300 8550 11000 8550
-Wire Wire Line
 	11500 8400 11500 8550
 Connection ~ 11500 8550
 Wire Wire Line
-	11500 8550 11300 8550
-Wire Wire Line
 	9600 7200 9600 8750
 Wire Wire Line
@@
 	11850 9650 11650 9650
 Wire Wire Line
-	9900 9650 9900 9500
-Wire Wire Line
 	11850 8550 11850 9650
 Wire Wire Line
 	10100 9500 10100 9650
-Connection ~ 10100 9650
-Wire Wire Line
-	10100 9650 9900 9650
-Wire Wire Line
-	10300 10750 10300 10600
-Wire Wire Line
-	10950 9500 10950 9650
-Connection ~ 10950 9650
 Wire Wire Line
 	11150 9500 11150 9650
 Connection ~ 11150 9650
 Wire Wire Line
-	11150 9650 10950 9650
-Wire Wire Line
-	11350 9500 11350 9650
-Connection ~ 11350 9650
-Wire Wire Line
-	11350 9650 11150 9650
-Wire Wire Line
 	11350 10200 11350 9850
 Wire Wire Line
@@
 Wire Wire Line
 	11650 9650 11650 10750
-Wire Wire Line
-	9900 10750 9900 10600
 Connection ~ 11650 9650
 Wire Wire Line
-	11650 9650 11350 9650
-Wire Wire Line
-	10100 9650 10300 9650
-Wire Wire Line
-	9900 10750 10100 10750
-Connection ~ 10300 10750
-Wire Wire Line
-	10300 10750 10950 10750
-Wire Wire Line
 	10100 10600 10100 10750
-Connection ~ 10100 10750
-Wire Wire Line
-	10100 10750 10300 10750
-Wire Wire Line
-	10950 10600 10950 10750
-Connection ~ 10950 10750
-Wire Wire Line
-	10950 10750 11150 10750
 Wire Wire Line
 	11150 10600 11150 10750
 Connection ~ 11150 10750
-Wire Wire Line
-	11150 10750 11350 10750
-Wire Wire Line
-	11350 10600 11350 10750
-Connection ~ 11350 10750
-Wire Wire Line
-	11350 10750 11650 10750
 Wire Wire Line
 	8850 8400 8850 10000
@@
 Text Label 3050 4650 0    50   ~ 0
 MIC
-Wire Wire Line
-	10300 9500 10300 9650
-Connection ~ 10300 9650
-Wire Wire Line
-	10300 9650 10950 9650
 $Comp
 L Device:R R5
@@
 Wire Wire Line
 	7650 3300 7850 3300
+$Comp
+L Device:LED_BARG D20
+U 1 1 5E72EAEB
+P 11150 10400
+F 0 "D20" V 11196 10070 50  0000 R CNN
+F 1 "LED_RGB" V 11105 10070 50  0000 R CNN
+F 2 "BBS Components:LED_RGB_SMD_PLCC4_Reverse_XZMDKCBDDG45S" H 11150 10350 50  0001 C CNN
+F 3 "~" H 11150 10350 50  0001 C CNN
+	1    11150 10400
+	0    -1   1    0
+$EndComp
+$Comp
+L Device:LED_BARG D18
+U 1 1 5E789449
+P 10100 10400
+F 0 "D18" V 10146 10070 50  0000 R CNN
+F 1 "LED_RGB" V 10055 10070 50  0000 R CNN
+F 2 "BBS Components:LED_RGB_SMD_PLCC4_Reverse_XZMDKCBDDG45S" H 10100 10350 50  0001 C CNN
+F 3 "~" H 10100 10350 50  0001 C CNN
+	1    10100 10400
+	0    -1   1    0
+$EndComp
+$Comp
+L Device:LED_BARG D10
+U 1 1 5E7D3287
+P 11500 8200
+F 0 "D10" V 11546 7870 50  0000 R CNN
+F 1 "LED_RGB" V 11455 7870 50  0000 R CNN
+F 2 "BBS Components:LED_RGB_SMD_PLCC4_Reverse_XZMDKCBDDG45S" H 11500 8150 50  0001 C CNN
+F 3 "~" H 11500 8150 50  0001 C CNN
+	1    11500 8200
+	0    -1   1    0
+$EndComp
+$Comp
+L Device:LED_BARG D14
+U 1 1 5E7D3281
+P 10800 8200
+F 0 "D14" V 10846 7870 50  0000 R CNN
+F 1 "LED_RGB" V 10755 7870 50  0000 R CNN
+F 2 "BBS Components:LED_RGB_SMD_PLCC4_Reverse_XZMDKCBDDG45S" H 10800 8150 50  0001 C CNN
+F 3 "~" H 10800 8150 50  0001 C CNN
+	1    10800 8200
+	0    -1   1    0
+$EndComp
+Text Label 11850 7650 0    50   ~ 0
+ALL_SEG
+$Comp
+L Device:LED_BARG D24
+U 1 1 5DC39FA4
+P 10100 8200
+F 0 "D24" V 10146 7870 50  0000 R CNN
+F 1 "LED_RGB" V 10055 7870 50  0000 R CNN
+F 2 "BBS Components:LED_RGB_SMD_PLCC4_Reverse_XZMDKCBDDG45S" H 10100 8150 50  0001 C CNN
+F 3 "~" H 10100 8150 50  0001 C CNN
+	1    10100 8200
+	0    -1   1    0
+$EndComp
+Wire Wire Line
+	10100 8400 10100 8550
+Wire Wire Line
+	10100 8550 10800 8550
+Wire Wire Line
+	10800 8550 11500 8550
+Wire Wire Line
+	11500 8550 11850 8550
+Wire Wire Line
+	11150 9650 11650 9650
+$Comp
+L Device:LED_BARG D11
+U 1 1 5E7108CE
+P 10100 9300
+F 0 "D11" V 10146 8970 50  0000 R CNN
+F 1 "LED_RGB" V 10055 8970 50  0000 R CNN
+F 2 "BBS Components:LED_RGB_SMD_PLCC4_Reverse_XZMDKCBDDG45S" H 10100 9250 50  0001 C CNN
+F 3 "~" H 10100 9250 50  0001 C CNN
+	1    10100 9300
+	0    -1   1    0
+$EndComp
+$Comp
+L Device:LED_BARG D15
+U 1 1 5E6D21EF
+P 11150 9300
+F 0 "D15" V 11196 8970 50  0000 R CNN
+F 1 "LED_RGB" V 11105 8970 50  0000 R CNN
+F 2 "BBS Components:LED_RGB_SMD_PLCC4_Reverse_XZMDKCBDDG45S" H 11150 9250 50  0001 C CNN
+F 3 "~" H 11150 9250 50  0001 C CNN
+	1    11150 9300
+	0    -1   1    0
+$EndComp
+Wire Wire Line
+	10100 9650 11150 9650
+Wire Wire Line
+	10100 10750 11150 10750
+Wire Wire Line
+	11150 10750 11650 10750
 $EndSCHEMATC

Commit message: new board RGB LED controll and 7-seg digits
Parts:
- removed C11: 10uF, Capacitors_SMD:C_0603_HandSoldering, symbol Device:C
- removed C7, C8: 22uF, Capacitors_SMD:C_0603_HandSoldering, symbol Device:C
- removed D1, D12, D13, D16, D17, D19, D2, D21, D22, D3, D4, D5, D6, D7, D8, D9: D, Diodes_SMD:D_SOD-523, symbol Device:D
- removed D18, D20, D24: LED_RGB, BBS Components:LED_RGB_SMD_PLCC4_Reverse_XZMDKCBDDG45S, symbol Device:LED_BARG
- removed D23: 7SegmentLED_ACDA02, BBS Components:7SegmentLED_ACDA02, symbol egdab:7SegmentLED_ACDA02
- removed J1: Audio-Jack-2_Switch, BBS Components:sj2-35852b-smt, symbol synthrotek2:Audio-Jack-2_Switch
- removed R7: 10K, Resistors_SMD:R_0603_HandSoldering, symbol Device:R
- removed RV5: R_POT, Potentiometers:Potentiometer_Trimmer_Suntan_TSR-3386P_Horizontal, symbol Device:R_POT
- removed SW1: SW_DIP_x12, Buttons_Switches_SMD:SW_DIP_x12_W8.61mm_Slide_LowProfile, symbol Switch:SW_DIP_x12
- removed SW3, SW4, SW5: SW_Push, BBS Components:SW_SPST_SMD_3_6, symbol Switch:SW_Push
- removed U4: CAP1296, Housings_SOIC:SOIC-14_3.9x8.7mm_Pitch1.27mm, symbol Sensor_Touch:CAP1206-x-SL
- added D1, D12, D13, D16, D2, D3, D4, D5, D6, D7, D8, D9: LED_RGB, BBS Components:LED_RGB_SMD_PLCC4_Reverse_XZMDKCBDDG45S, symbol Device:LED_BARG
- added D17: 7SegmentLED_ACSC02, BBS Components:7SegmentLED_ACSC02, symbol egdab:7SegmentLED_ACSC02
- added R11, R12, R13: 10K, Resistors_SMD:R_0603_HandSoldering, symbol Device:R
- added R7: R_PHOTO, LEDs:LED_D4.0mm, symbol Device:R_PHOTO
- added R8, R9: 4K7, Resistors_SMD:R_0603_HandSoldering, symbol Device:R
- added SW1: SW_DIP_x04, Buttons_Switches_SMD:SW_DIP_x4_W8.61mm_Slide_LowProfile, symbol Switch:SW_DIP_x04
Connections:
- net labels added: PHOTO, P_CHROMA+, P_CHROMA-, P_LUMA, P_TIME
- net labels removed: ALL_SEG, KEYB, MIC, POT1, POT2, POT3, POT4, POT5, TOUCH1, TOUCH2, TOUCH_GUARD, TOUCH_PROX
- wire segments 477 -> 139
Other:
- note removed: "TODO share voltage divider and capacitor between audio sources"
- moved on the sheet: MK1, R2, RV1, RV2, SW2, U3
