File: kicad/egdab.kicad_pcb (KiCad board)
At the start: 2 copper layers, 57 parts, among them J2 Conn_02x03_Counter_Clockwise, J3 Conn_02x10_Counter_Clockwise, SW1 SW_DIP_x12, U1 ATtiny1606-S, U2 AS1115-BSST, U3 LM35-D, U4 CAP1296

Commit message: Big things
Parts:
- removed C12: 10uF, Capacitors_SMD:C_0603_HandSoldering
- removed R8, R9: 10K, Resistors_SMD:R_0603_HandSoldering
- added D23: 7SegmentLED_ACDA02, BBS Components:7SegmentLED_ACDA02, F.Cu at (188.0, 105.8)
- added D24: LED_RGB, LEDs:LED_RGB_PLCC-6, B.Cu at (213.5, 125.5)
- added G***: LOGO, BBS Components:silkscreen-1, F.Cu at (180.0, 97.0)
- added G***: LOGO, BBS Components:soldermask-1, F.Cu at (180.0, 97.0)
- added SW2: SW_Push, BBS Components:SW_SPST_SMD_3_6, B.Cu at (204.5, 99.8)
- added SW3: SW_Push, BBS Components:SW_SPST_SMD_3_6, B.Cu at (204.5, 92.2)
- added SW4: SW_Push, BBS Components:SW_SPST_SMD_3_6, B.Cu at (204.5, 103.5)
- added SW5: SW_Push, BBS Components:SW_SPST_SMD_3_6, B.Cu at (204.5, 96.0)
- BT1, D1, D10, D11, D12, D13, D14, D15, D16, D17, D18, D19, D2, D20, D21, D22, D3, D4, D5, D6, D7, D8, D9, R2, SW1, U1, U2, U4: moved to B.Cu
- J2: footprint Pin_Headers:Pin_Header_Straight_2x03_Pitch2.54mm -> BBS Components:Header_SMD_vertical_passthrough_02x03; moved to B.Cu
- J3: value Conn_02x10_Counter_Clockwise -> Conn_02x04_Counter_Clockwise; footprint Pin_Headers:Pin_Header_Angled_2x10_Pitch2.54mm -> BBS Components:Header_SMD_vertical_passthrough_02x04; moved to B.Cu
- moved U3 168.6 mm to (174.0, 105.8)
- moved D20 151.1 mm to (206.0, 82.5)
- moved R2 149.3 mm to (184.0, 138.4), turned to 270 degrees
- moved U1 126.2 mm to (147.8, 89.2), turned to 90 degrees
- moved U4 125.5 mm to (202.5, 118.8)
- moved D8 110.5 mm to (176.5, 85.8)
- moved D11 108.5 mm to (162.0, 90.0), turned to 180 degrees
- moved D13 107.5 mm to (179.0, 83.5)
- moved D16 103.1 mm to (179.0, 77.5)
- moved D18 100.6 mm to (195.0, 90.8), turned to 270 degrees
- moved D9 99.4 mm to (179.0, 76.0)
- moved D7 97.4 mm to (176.5, 82.8)
- moved D6 95.8 mm to (176.5, 79.8)
- moved D1 93.6 mm to (176.5, 76.8)
- moved D17 92.0 mm to (179.0, 74.5)
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Connections:
- net Net-(C11-Pad2) renamed /MIC
- net Net-(C9-Pad2) renamed /AUDIO
- net Net-(D1-Pad2) renamed /SEGDP
- net Net-(D12-Pad2) renamed /SEGG
- net Net-(D13-Pad2) renamed /SEGF
- net Net-(D16-Pad2) renamed /SEGE
- net Net-(D17-Pad2) renamed /SEGD
- net Net-(D19-Pad2) renamed /SEGC
- net Net-(D21-Pad2) renamed /SEGB
- net Net-(D22-Pad2) renamed /SEGA
- net Net-(R1-Pad2) renamed /AS1115_ISET
- net Net-(RV1-Pad2) renamed /POT1
- net Net-(RV2-Pad2) renamed /POT2
- net Net-(RV3-Pad2) renamed /POT3
- net Net-(RV4-Pad2) renamed /POT4
- net Net-(RV5-Pad2) renamed /POT5
- net Net-(SW1-Pad1) renamed /KEYA
- net Net-(SW1-Pad10) renamed /KEYB
- net Net-(U1-Pad4) renamed /TEMP
- BT1 pad 1: +3V0 -> Net-(BT1-Pad1)
- C1 pad 1: +3V0 -> Net-(BT1-Pad1)
- C2 pad 1: +3V0 -> Net-(BT1-Pad1)
- C3 pad 1: +3V0 -> Net-(BT1-Pad1)
- C4 pad 1: +3V0 -> Net-(BT1-Pad1)
- C5 pad 1: +3V0 -> Net-(BT1-Pad1)
- C6 pad 1: +3V0 -> Net-(BT1-Pad1)
- C7 pad 1: +3V0 -> Net-(BT1-Pad1)
- C8 pad 1: +3V0 -> Net-(BT1-Pad1)
- D10 pad 1: Net-(D10-Pad1) -> /DIG4
- D10 pad 2: Net-(D10-Pad2) -> /DIG3
- D10 pad 3: Net-(D10-Pad3) -> /DIG2
- D10 pad 5: Net-(D10-Pad5) -> Net-(D10-Pad4)
- D10 pad 6: Net-(D10-Pad6) -> Net-(D10-Pad4)
- D11 pad 1: Net-(D11-Pad1) -> /DIG7
- D11 pad 2: Net-(D11-Pad2) -> /DIG6
- D11 pad 3: Net-(D11-Pad3) -> /DIG5
- D11 pad 4: Net-(D11-Pad4) -> Net-(D10-Pad4)
- D11 pad 5: Net-(D11-Pad5) -> Net-(D10-Pad4)
- D11 pad 6: Net-(D11-Pad6) -> Net-(D10-Pad4)
- D12 pad 1: Net-(D12-Pad1) -> Net-(D10-Pad4)
- D13 pad 1: Net-(D12-Pad1) -> Net-(D10-Pad4)
- D14 pad 1: Net-(D10-Pad6) -> /DIG4
- D14 pad 2: Net-(D10-Pad5) -> /DIG3
- D14 pad 3: Net-(D10-Pad4) -> /DIG2
- D14 pad 4: Net-(D12-Pad1) -> Net-(D10-Pad4)
- D14 pad 5: Net-(D12-Pad1) -> Net-(D10-Pad4)
- D14 pad 6: Net-(D12-Pad1) -> Net-(D10-Pad4)
- D15 pad 1: Net-(D11-Pad6) -> /DIG7
- D15 pad 2: Net-(D11-Pad5) -> /DIG6
- D15 pad 3: Net-(D11-Pad4) -> /DIG5
- D15 pad 4: Net-(D15-Pad4) -> Net-(D10-Pad4)
- D15 pad 5: Net-(D15-Pad5) -> Net-(D10-Pad4)
- D15 pad 6: Net-(D15-Pad6) -> Net-(D10-Pad4)
- D16 pad 1: Net-(D12-Pad1) -> Net-(D10-Pad4)
- D17 pad 1: Net-(D12-Pad1) -> Net-(D10-Pad4)
- D18 pad 1: Net-(D15-Pad6) -> /DIG7
- D18 pad 2: Net-(D15-Pad5) -> /DIG6
- D18 pad 3: Net-(D15-Pad4) -> /DIG5
- D18 pad 4: Net-(D18-Pad4) -> Net-(D10-Pad4)
- D18 pad 5: Net-(D18-Pad5) -> Net-(D10-Pad4)
- D18 pad 6: Net-(D18-Pad6) -> Net-(D10-Pad4)
- D19 pad 1: Net-(D12-Pad1) -> Net-(D10-Pad4)
- D20 pad 1: Net-(D18-Pad6) -> /DIG7
- D20 pad 2: Net-(D18-Pad5) -> /DIG6
- D20 pad 3: Net-(D18-Pad4) -> /DIG5
- D20 pad 4: Net-(D12-Pad1) -> Net-(D10-Pad4)
- D20 pad 5: Net-(D12-Pad1) -> Net-(D10-Pad4)
- D20 pad 6: Net-(D12-Pad1) -> Net-(D10-Pad4)
- D21 pad 1: Net-(D12-Pad1) -> Net-(D10-Pad4)
- D22 pad 1: Net-(D12-Pad1) -> Net-(D10-Pad4)
- D6 pad 1: Net-(D1-Pad1) -> Net-(D6-Pad1)
- D7 pad 1: Net-(D2-Pad1) -> Net-(D7-Pad1)
- D8 pad 1: Net-(D3-Pad1) -> Net-(D8-Pad1)
- D9 pad 1: Net-(D12-Pad1) -> Net-(D10-Pad4)
- J3 pad 1: RESET -> GND
- J3 pad 2: SPI_SS -> GND
- J3 pad 3: SPI_MOSI -> UI_INTERRUPT
- J3 pad 4: SPI_MISO -> SPI_SS
- J3 pad 6: I2C_SCL -> SPI_MISO
- J3 pad 7: I2C_SDA -> SPI_MOSI
- J3 pad 8: PB3 -> RESET
- R10 pad 2: Net-(C12-Pad2) -> Net-(C10-Pad2)
- SW1 pad 17: Net-(D3-Pad1) -> Net-(D8-Pad1)
- SW1 pad 18: Net-(D2-Pad1) -> Net-(D7-Pad1)
- SW1 pad 19: Net-(D1-Pad1) -> Net-(D6-Pad1)
- U2 pad 10: Net-(D11-Pad1) -> /DIG7
- U2 pad 2: Net-(U2-Pad2) -> /DIG0
- U2 pad 3: Net-(U2-Pad3) -> /DIG1
- U2 pad 4: Net-(D10-Pad3) -> /DIG2
- U2 pad 5: Net-(D10-Pad2) -> /DIG3
- U2 pad 7: Net-(D10-Pad1) -> /DIG4
- U2 pad 8: Net-(D11-Pad3) -> /DIG5
- U2 pad 9: Net-(D11-Pad2) -> /DIG6
Routing:
- net UI_INTERRUPT: track 0.00 -> 142.2 mm, vias 0 -> 2
- net I2C_SDA: track 0.00 -> 136.5 mm, vias 0 -> 7
- net Net-(D10-Pad4): track 0.00 -> 127.4 mm, vias 0 -> 6
- net I2C_SCL: track 0.00 -> 106.9 mm, vias 0 -> 8
- net /POT5: track 0.00 -> 99.2 mm, vias 0 -> 4
- net /POT3: track 0.00 -> 95.2 mm, vias 0 -> 2
- net /POT2: track 0.00 -> 87.5 mm, vias 0 -> 2
- net /POT1: track 0.00 -> 79.6 mm, vias 0 -> 2
- net /POT4: track 0.00 -> 75.8 mm, vias 0 -> 2
- net /DIG5: track 0.00 -> 74.4 mm, vias 0 -> 5
- net /SEGD: track 0.00 -> 73.3 mm, vias 0 -> 4
- net /KEYB: track 0.00 -> 72.4 mm, vias 0 -> 2
- net /DIG6: track 0.00 -> 72.0 mm, vias 0 -> 5
- net /DIG7: track 0.00 -> 69.0 mm, vias 0 -> 5
- net SPI_SCK: track 0.00 -> 68.6 mm, vias 0 -> 2
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- added copper zone on In2.Cu, net GND
Other:
- board outline added: 93.4 x 99.4 mm
- copper layers 2 -> 4
- rule via_min_drill: 0.3 -> 0.2
- rule via_min_size: 0.4 -> 0.45

Commit message: PCB layout progress
Parts:
- added SW6: SW_SPST, Digikey:Switch_Slide_JS202011SCQN, B.Cu at (198.0, 133.8)
- C1, C2, C3, C4, C5, C7, C8, R1: moved to B.Cu
- moved C3 102.7 mm to (202.5, 113.8)
- moved C8 97.0 mm to (189.2, 126.0), turned to 180 degrees
- moved C4 92.9 mm to (189.2, 128.5), turned to 180 degrees
- moved C5 89.3 mm to (189.2, 127.2), turned to 180 degrees
- moved C7 89.1 mm to (189.2, 124.8), turned to 180 degrees
- moved R1 69.0 mm to (181.0, 87.0)
- moved C2 65.5 mm to (184.0, 73.8), turned to 180 degrees
- moved C6 62.9 mm to (174.0, 109.0), turned to 180 degrees
- moved C1 47.9 mm to (156.2, 93.5), turned to 90 degrees
- moved R2 12.3 mm to (180.0, 126.8), turned to 90 degrees
- moved U2 0.75 mm to (185.0, 79.2)
Connections:
- BT1 pad 1: Net-(BT1-Pad1) -> /BAT+
- C1 pad 1: Net-(BT1-Pad1) -> +3V0
- C2 pad 1: Net-(BT1-Pad1) -> +3V0
- C3 pad 1: Net-(BT1-Pad1) -> +3V0
- C4 pad 1: Net-(BT1-Pad1) -> +3V0
- C5 pad 1: Net-(BT1-Pad1) -> +3V0
- C6 pad 1: Net-(BT1-Pad1) -> +3V0
- C7 pad 1: Net-(BT1-Pad1) -> +3V0
- C8 pad 1: Net-(BT1-Pad1) -> +3V0
- D10 pad 1: /DIG4 -> /DIG2
- D10 pad 2: /DIG3 -> /DIG1
- D10 pad 3: /DIG2 -> /DIG0
- D14 pad 1: /DIG4 -> /DIG2
- D14 pad 2: /DIG3 -> /DIG1
- D14 pad 3: /DIG2 -> /DIG0
- D23 pad 13: /DIG0 -> /DIG3
- D23 pad 18: /DIG1 -> /DIG4
- D23 pad 3: /DIG1 -> /DIG4
- D23 pad 8: /DIG0 -> /DIG3
- D24 pad 1: /DIG4 -> /DIG2
- D24 pad 2: /DIG3 -> /DIG1
- D24 pad 3: /DIG2 -> /DIG0
Routing:
- net +3V0: track 3.88 -> 198.9 mm, vias 0 -> 15
- net /DIG2: track 0.00 -> 157.3 mm, vias 0 -> 5
- net /DIG1: track 19.6 -> 155.2 mm, vias 2 -> 5
- net /DIG0: track 14.4 -> 147.9 mm, vias 1 -> 5
- net Net-(D10-Pad4): track 127.4 -> 258.7 mm, vias 6 -> 9
- net /BAT+: track 0.00 -> 83.5 mm, vias 0 -> 2
- net /DIG4: track 0.00 -> 62.9 mm, vias 0 -> 3
- net /DIG3: track 0.00 -> 47.1 mm, vias 0 -> 2
- net GND: track 8.00 -> 49.8 mm, vias 20 -> 31
- net /AS1115_ISET: track 0.40 -> 4.38 mm
- net UI_INTERRUPT: track 142.2 -> 144.1 mm
- net Net-(R2-Pad1): track 48.5 -> 50.3 mm, vias 3 -> 2
- net /SEGA: track 54.2 -> 55.5 mm
- net /SEGF: track 49.7 -> 50.9 mm
- net /SEGG: track 52.0 -> 53.1 mm
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Other:
- net class Bat+ added: clearance 0.2, trace_width 1, via_dia 0.8, via_drill 0.4
- net class Default: via_dia 0.8 -> 0.45; via_drill 0.4 -> 0.2
- net class Power added: clearance 0.2, trace_width 0.5, via_dia 0.45, via_drill 0.2

Commit message: Draft 1 may be complete
Parts:
- added J1: Audio-Jack-2_Switch, BBS Components:sj2-35852b-smt, B.Cu at (216.8, 85.2)
- added MK1: Microphone, BBS Components:spv1840l45h-b, B.Cu at (209.0, 69.8)
- C10, C11, C9, R10, R3, R4, R5, R6, R7: moved to B.Cu
- D10, D11, D14, D15, D18, D20, D24: footprint LEDs:LED_RGB_PLCC-6 -> BBS Components:plcc_6_reverse_smd_rgb_led
- moved R10 105.8 mm to (205.8, 73.2), turned to 270 degrees
- moved C9 93.2 mm to (220.2, 78.5), turned to 180 degrees
- moved R7 92.1 mm to (211.0, 71.0), turned to 270 degrees
- moved R3 91.4 mm to (217.2, 80.8), turned to 180 degrees
- moved R4 88.1 mm to (210.0, 77.5), turned to 90 degrees
- moved C10 87.2 mm to (211.0, 74.5), turned to 180 degrees
- moved R5 86.7 mm to (213.0, 76.2)
- moved R6 85.0 mm to (205.8, 77.5), turned to 90 degrees
- moved C11 79.7 mm to (208.5, 72.2), turned to 180 degrees
- moved D14 1.12 mm to (148.5, 124.8)
- moved C4 0.75 mm to (189.2, 129.2)
- moved C3 0.50 mm to (202.5, 113.2)
- moved C5 0.50 mm to (189.2, 127.8)
- moved D11 0.50 mm to (162.0, 89.5)
- moved C6 0.25 mm to (174.0, 109.2)
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Routing:
- net /AUDIO: track 0.00 -> 96.3 mm, vias 0 -> 4
- net /MIC: track 0.00 -> 91.5 mm, vias 0 -> 2
- net TOUCH_GUARD: track 0.00 -> 70.0 mm, vias 0 -> 3
- net TOUCH1: track 0.00 -> 48.3 mm, vias 0 -> 2
- net +3V0: track 198.9 -> 240.1 mm, vias 15 -> 16
- net GND: track 49.8 -> 66.1 mm, vias 31 -> 33
- net Net-(C10-Pad2): track 0.00 -> 10.2 mm
- net TOUCH_PROX: track 0.00 -> 9.52 mm, vias 0 -> 1
- net Net-(C9-Pad1): track 0.00 -> 6.16 mm
- net TOUCH2: track 0.00 -> 4.11 mm, vias 0 -> 1
- net Net-(D10-Pad4): track 258.7 -> 262.5 mm
- net Net-(C11-Pad1): track 0.00 -> 3.37 mm
- net SPI_SS: track 64.4 -> 67.5 mm
- net SPI_MOSI: track 65.4 -> 68.3 mm
- net SPI_MISO: track 68.1 -> 70.7 mm
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- added copper zone on In2.Cu, net TOUCH1
- added copper zone on In2.Cu, net TOUCH2
- added copper zone on In2.Cu, net TOUCH_GUARD
- added copper zone on In2.Cu, net TOUCH_PROX
Other:
- board text added: "+3V"
- board text added: "A"
- board text added: "B"
- board text added: "C"
- board text added: "D"
- board text added: "E"
- board text added: "F"
- board text added: "G"
- board text added: "GND"
- board text added: "H"
- board text added: "Happy Birthday Brooke! 2019"
- board text added: "I"
- board text added: "J"
- board text added: "K"
- board text added: "L"
- board text added: "MISO"
- board text added: "MOSI"
- board text added: "PB2"
- board text added: "PB3"
- board text added: "RST"
- board text added: "SCK"
- board text added: "SCL"
- board text added: "SDA"
- board text added: "SS"
- board text added: "UI_INT"

Commit message: v2 PCB in progress
- board version added to silk
- use actual reverse mount RGB LEDs
- invert lower petal soldermask
Parts:
- D10, D11, D14, D15, D18, D20, D24: footprint BBS Components:plcc_6_reverse_smd_rgb_led -> BBS Components:LED_RGB_SMD_PLCC4_Reverse_XZMDKCBDDG45S
- G***: footprint BBS Components:soldermask-1 -> BBS Components:soldermask-2
Connections:
- D10 pad 1: /DIG2 -> /DIG0
- D10 pad 2: /DIG1 -> /ALL_SEG
- D10 pad 3: /DIG0 -> /DIG2
- D10 pad 4: Net-(D10-Pad4) -> /DIG1
- D11 pad 1: /DIG7 -> /DIG5
- D11 pad 2: /DIG6 -> /ALL_SEG
- D11 pad 3: /DIG5 -> /DIG7
- D11 pad 4: Net-(D10-Pad4) -> /DIG6
- D12 pad 1: Net-(D10-Pad4) -> /ALL_SEG
- D13 pad 1: Net-(D10-Pad4) -> /ALL_SEG
- D14 pad 1: /DIG2 -> /DIG0
- D14 pad 2: /DIG1 -> /ALL_SEG
- D14 pad 3: /DIG0 -> /DIG2
- D14 pad 4: Net-(D10-Pad4) -> /DIG1
- D15 pad 1: /DIG7 -> /DIG5
- D15 pad 2: /DIG6 -> /ALL_SEG
- D15 pad 3: /DIG5 -> /DIG7
- D15 pad 4: Net-(D10-Pad4) -> /DIG6
- D16 pad 1: Net-(D10-Pad4) -> /ALL_SEG
- D17 pad 1: Net-(D10-Pad4) -> /ALL_SEG
- D18 pad 1: /DIG7 -> /DIG5
- D18 pad 2: /DIG6 -> /ALL_SEG
- D18 pad 3: /DIG5 -> /DIG7
- D18 pad 4: Net-(D10-Pad4) -> /DIG6
- D19 pad 1: Net-(D10-Pad4) -> /ALL_SEG
- D20 pad 1: /DIG7 -> /DIG5
- D20 pad 2: /DIG6 -> /ALL_SEG
- D20 pad 3: /DIG5 -> /DIG7
- D20 pad 4: Net-(D10-Pad4) -> /DIG6
- D21 pad 1: Net-(D10-Pad4) -> /ALL_SEG
- D22 pad 1: Net-(D10-Pad4) -> /ALL_SEG
- D24 pad 1: /DIG2 -> /DIG0
- D24 pad 2: /DIG1 -> /ALL_SEG
- D24 pad 3: /DIG0 -> /DIG2
- D24 pad 4: Net-(D10-Pad4) -> /DIG1
- D9 pad 1: Net-(D10-Pad4) -> /ALL_SEG
Routing:
- net Net-(D10-Pad4): track 262.5 -> 0.00 mm, vias 9 -> 0
- net /ALL_SEG: track 0.00 -> 235.8 mm, vias 0 -> 11
- net /DIG6: track 70.4 -> 100.1 mm
- net /DIG0: track 148.2 -> 175.8 mm, vias 5 -> 6
- net /DIG1: track 155.6 -> 171.4 mm, vias 5 -> 6
- net /DIG5: track 73.4 -> 86.4 mm, vias 5 -> 4
- net /DIG2: track 158.6 -> 157.1 mm, vias 5 -> 6
- net /DIG7: track 67.6 -> 68.3 mm
Other:
- board text added: "BBS 2019 v2"
- board text added: "Happy Birthday Brooke!"
- board text removed: "Happy Birthday Brooke! 2019"
